Commit message: update

File: Controller/project_starter/panda/Urdf_files/GEN3_URDF_V12.urdf (robot description, URDF)
Before this commit: robot kinova, 9 links, 8 joints
Links:
- link link0: geometry visual mesh filename=../../urdf_models/mmp_panda/meshes/base_link.obj
- link link1: geometry visual mesh filename=../../urdf_models/mmp_panda/meshes/Shoulder_Link.obj
- link link2: geometry visual mesh filename=../../urdf_models/mmp_panda/meshes/HalfArm1_Link.obj
- link link3: geometry visual mesh filename=../../urdf_models/mmp_panda/meshes/HalfArm2_Link.obj
- link link4: geometry collision mesh filename=../../urdf_models/mmp_panda/meshes/ForeArm_Link.obj; visual mesh filename=../../urdf_models/mmp_panda/meshes/ForeArm_Link.obj
- link link5: geometry collision mesh filename=../../urdf_models/mmp_panda/meshes/SphericalWrist1_Link.obj; visual mesh filename=../../urdf_models/mmp_panda/meshes/SphericalWrist1_Link.obj
- link link6: geometry collision mesh filename=../../urdf_models/mmp_panda/meshes/SphericalWrist2_Link.obj; visual mesh filename=../../urdf_models/mmp_panda/meshes/SphericalWrist2_Link.obj
- link link7: geometry collision mesh filename=../../urdf_models/mmp_panda/meshes/bracelet_no_vision_link.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; visual mesh filename=../../urdf_models/mmp_panda/meshes/bracelet_no_vision_link.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
